Commit message: Subiendo Reporte de Practica 1

File: urdf/robot_rrr.urdf (robot description, URDF)
Before this commit: robot robot, 4 links, 3 joints
Links:
- removed link arm_link
- removed link forearm_link
- removed link shoulder_link
- added link link2; visual box size=0.4 0.06 0.06
- added link link2_punta
- added link link3; visual cylinder length=0.3 radius=0.02
- added link link_brazo_azul; visual box size=0.4 0.08 0.08
- added link link_columna; visual cylinder length=0.6 radius=0.05
- link base_link: geometry visual cylinder length=0.1 radius=0.2
Joints:
- removed joint arm_joint
- removed joint forearm_joint
- removed joint shoulder_joint
- added joint joint1: type revolute, parent base_link, child link_columna, origin xyz=0 0 0.1 rpy=0 0 0, axis 0 0 1, limit lower=-3.1416 upper=3.1416 effort=10.0 velocity=1.0
- added joint joint2: type revolute, parent link_brazo_azul, child link2, origin xyz=0.4 0 0.07 rpy=0 0 0, axis 0 0 1, limit lower=-2.5 upper=2.5 effort=10.0 velocity=1.0
- added joint joint3: type prismatic, parent link2_punta, child link3, origin xyz=0 0 0 rpy=0 0 0, axis 0 0 1, limit lower=-0.25 upper=0.0 effort=10.0 velocity=1.0
- added joint junta_fija_L: type fixed, parent link_columna, child link_brazo_azul, origin xyz=0 0 0.6 rpy=0 0 0
- added joint junta_referencia_verde: type fixed, parent link2, child link2_punta, origin xyz=0.4 0 0 rpy=0 0 0
